File: pcb/ESPlant.kicad_pcb (KiCad board)
At the start: 2 copper layers, 43 x 23 mm, 25 parts, among them J1 Power, J2 TAG, J3 PUMP, J4 Soil Moisture, Q1 Q_NPN_BEC, Q2 Pump Driver, U1 ESP32-WROOM-32, U2 Si7021-A20, U3 LD1117S33TR_SOT223

Commit message: Flipping batter positive and negative pins and added '+' symbol to resolve ambiguity during assembly
Parts:
- Q1: value Q_NPN_BEC -> MMBT2222ALT1G
- R3: value R -> 33k
- R4: value R -> 51k
Connections:
- J1 pad 1: GNDREF -> +BATT
- J1 pad 2: +BATT -> GNDREF
Routing:
- net +BATT: track 12.4 -> 14.1 mm
- net GNDREF: track 8.89 -> 10.4 mm
Other:
- board text added: "+"
- board text added: "ESPlant - Rev 0.3b Sandor Labs 2020-08"
- board text removed: "ESPlant - Rev 0.2 Ed Sandor 2020-03"
Changed lines of the file:
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@@
   (general
     (thickness 1.6)
-    (drawings 5)
-    (tracks 164)
+    (drawings 6)
+    (tracks 170)
     (zones 0)
     (modules 25)
@@
       (effects (font (size 1 1) (thickness 0.15)) (justify mirror))
     )
-    (fp_text value Q_NPN_BEC (at 0 -2.5 270) (layer B.Fab)
+    (fp_text value MMBT2222ALT1G (at 0 -2.5 270) (layer B.Fab)
       (effects (font (size 1 1) (thickness 0.15)) (justify mirror))
     )
@@
       (effects (font (size 1 1) (thickness 0.15)) (justify mirror))
     )
-    (fp_text value R (at 0 -1.43 270) (layer B.Fab) hide
+    (fp_text value 51k (at 0 -1.43 270) (layer B.Fab) hide
       (effects (font (size 1 1) (thickness 0.15)) (justify mirror))
     )
@@
       (effects (font (size 1 1) (thickness 0.15)) (justify mirror))
     )
-    (fp_text value R (at 0 -1.43 270) (layer B.Fab) hide
+    (fp_text value 33k (at 0 -1.43 270) (layer B.Fab) hide
       (effects (font (size 1 1) (thickness 0.15)) (justify mirror))
     )
@@
     (fp_line (start -0.635 -1.27) (end 1.27 -1.27) (layer F.Fab) (width 0.1))
     (pad 2 thru_hole oval (at 0 2.54) (size 1.7 1.7) (drill 1) (layers *.Cu *.Mask)
+      (net 1 GNDREF))
+    (pad 1 thru_hole rect (at 0 0) (size 1.7 1.7) (drill 1) (layers *.Cu *.Mask)
       (net 6 +BATT))
-    (pad 1 thru_hole rect (at 0 0) (size 1.7 1.7) (drill 1) (layers *.Cu *.Mask)
-      (net 1 GNDREF))
     (model ${KISYS3DMOD}/Connector_PinHeader_2.54mm.3dshapes/PinHeader_1x02_P2.54mm_Vertical.wrl
       (at (xyz 0 0 0))
@@
     )
   )
-  (gr_text "ESPlant - Rev 0.2\nEd Sandor 2020-03" (at 149.5 91.25) (layer B.SilkS)
+  (gr_text + (at 172.75 91.25) (layer F.SilkS)
+    (effects (font (size 1.5 1.5) (thickness 0.3)))
+  )
+  (gr_text "ESPlant - Rev 0.3b\nSandor Labs 2020-08" (at 149.5 91.25) (layer B.SilkS)
     (effects (font (size 1.5 1.5) (thickness 0.3)) (justify mirror))
   )
@@
   (segment (start 146.573002 96.5) (end 136.96 96.5) (width 0.25) (layer B.Cu) (net 5))
   (segment (start 167.16 91.7) (end 167 91.7) (width 0.25) (layer F.Cu) (net 6))
-  (segment (start 171 95.54) (end 167.16 91.7) (width 0.25) (layer F.Cu) (net 6))
-  (segment (start 170.46 95.54) (end 171 95.54) (width 0.25) (layer F.Cu) (net 6))
-  (segment (start 170.29 96.25) (end 171 95.54) (width 0.25) (layer B.Cu) (net 6))
-  (segment (start 165 96.25) (end 170.29 96.25) (width 0.25) (layer B.Cu) (net 6))
+  (segment (start 170.46 95.54) (end 171 95.54) (width 0.25) (layer F.Cu) (net 1))
+  (segment (start 170.29 96.25) (end 171 95.54) (width 0.25) (layer B.Cu) (net 1))
+  (segment (start 171 91.9) (end 171 93) (width 0.25) (layer F.Cu) (net 6))
+  (segment (start 170.8 91.7) (end 171 91.9) (width 0.25) (layer F.Cu) (net 6))
+  (segment (start 167 91.7) (end 170.8 91.7) (width 0.25) (layer F.Cu) (net 6))
+  (segment (start 169 95.725) (end 169 96.25) (width 0.25) (layer B.Cu) (net 6))
+  (segment (start 169.9 93) (end 169 93.9) (width 0.25) (layer B.Cu) (net 6))
+  (segment (start 169 93.9) (end 169 95.725) (width 0.25) (layer B.Cu) (net 6))
+  (segment (start 171 93) (end 169.9 93) (width 0.25) (layer B.Cu) (net 6))
+  (segment (start 169 96.25) (end 165 96.25) (width 0.25) (layer B.Cu) (net 6))
   (via (at 160 97.5) (size 0.8) (drill 0.4) (layers F.Cu B.Cu) (net 7))
   (segment (start 157.095 99) (end 157 99.095) (width 0.25) (layer F.Cu) (net 7))
